File: WeMos_Shield_Bricolabs/wemos-01.kicad_pcb (KiCad board)
At the start: 2 copper layers, 25.7 x 34.4 mm, 17 parts, among them J1 Conn_01x04, J2 Conn_01x01, P1 CONN_01X08, P2 CONN_01X08, U1 RFM95W-915S2

Commit message: Add some updates
Parts:
- removed the REF** at (140.5, 91.6)
- added G***: LOGO, varios:bricolabs8, B.Cu at (139.7, 91.2)
- moved svg2mod 0.76 mm to (139.7, 94.9)
