File: WeMos_Shield_Greynaga/wemos-01.kicad_pcb (KiCad board)
At the start: 2 copper layers, 25.7 x 34.4 mm, 17 parts, among them J1 Conn_01x04, J2 Conn_01x01, P1 CONN_01X08, P2 CONN_01X08, U1 RFM95W-915S2

Commit message: Add gitignore
Parts:
- moved svg2mod 0.20 mm to (139.9, 95.6)
Other:
- board text added: "DI00"
- board text added: "DI01"
- board text added: "MISO"
- board text added: "MOSI"
- board text added: "NSS"
- board text added: "SCK"

Commit message: Updates
Parts:
- removed GBSilk*** (x2): LOGO, varios:greynaga6-2-Mask
- removed GS*** (x2): v, varios:greynaga6-2-Cooper
- removed REF**: KiCad-Logo2_6mm_SilkScreen, Symbol:KiCad-Logo2_6mm_SilkScreen
- removed REF**: OSHW-Logo2_9.8x8mm_SilkScreen, Symbol:OSHW-Logo2_9.8x8mm_SilkScreen
- removed REF**: OSHW-Logo2_7.3x6mm_SilkScreen, Symbol:OSHW-Logo2_7.3x6mm_SilkScreen
- removed svg2mod: G***, Varios:ttn_logoCu1
- removed svg2mod: G***, Varios:ttn_logo3
- added U2: Kicad-Logo2, WeMos_Shield_Greynaga:KiCad-Logo2_6mm_SilkScreen, B.Cu at (140.0, 101.0)
- added U3: OSHW_2_7, WeMos_Shield_Greynaga:OSHW-Logo2_7.3x6mm_SilkScreen, F.Cu at (130.5, 83.3)
- added U4: OSHW_2_9, WeMos_Shield_Greynaga:OSHW-Logo2_9.8x8mm_SilkScreen, B.Cu at (140.2, 93.9)
- added U5: Firma_Cooper, WeMos_Shield_Greynaga:greynaga6-2-Cooper, B.Cu at (134.9, 110.9)
- added U5: Firma_Cooper, WeMos_Shield_Greynaga:greynaga6-2-Cooper, F.Cu at (134.9, 111.1)
- added U6: Firma_Mask, WeMos_Shield_Greynaga:greynaga6-2-Mask, B.Cu at (134.9, 110.9)
- added U6: Firma_Mask, WeMos_Shield_Greynaga:greynaga6-2-Mask, F.Cu at (134.9, 111.1)
- added U7: TTN_Silk, WeMos_Shield_Greynaga:ttn_logo3, F.Cu at (139.8, 95.4)
- added U8: TTN_Cooper, WeMos_Shield_Greynaga:ttn_logoCu1, B.Cu at (132.0, 83.5)
- A2: footprint Cats_ArduinoShieldLoRa:SMA_EDGELAUNCH_UFL_WeMos_Lora -> WeMos_Shield_Greynaga:SMA_EDGELAUNCH_UFL_WeMos_Lora
- C1, C2: footprint Capacitor_SMD:C_0805_2012Metric_Pad1.29x1.40mm_HandSolder -> WeMos_Shield_Greynaga:C_0805_2012Metric_Pad1.29x1.40mm_HandSolder
- J1: footprint Connector_PinSocket_2.54mm:PinSocket_1x04_P2.54mm_WeMos -> WeMos_Shield_Greynaga:PinSocket_1x04_P2.54mm_WeMos
- J2: footprint Connector_PinSocket_2.54mm:PinSocket_1x01_P2.54mm_WeMos -> WeMos_Shield_Greynaga:PinSocket_1x01_P2.54mm_WeMos
- P1, P2: footprint D1_mini:D1_mini_Pin_Header -> WeMos_Shield_Greynaga:D1_mini_Pin_Header
- U1: footprint RF_Module:HOPERF_RFM9XW_SMD_WeMos -> WeMos_Shield_Greynaga:HOPERF_RFM9XW_SMD_WeMos
Connections:
- U1 pad 6: /RST -> Net-(U1-Pad6)
Routing:
- net /RST: track 24.2 -> 0.22 mm, vias 1 -> 0
Other:
- board text added: "D0"
- board text added: "D1"
- board text added: "D2"
- board text added: "D5"
- board text added: "D6"
- board text added: "D7"
- board text added: "io2"
- board text added: "io3"
- board text added: "io4"
- board text added: "io5"
- board text removed: "G2"
- board text removed: "G3"
- board text removed: "G4"
- board text removed: "G5"
